File: INRUSH_CURRENT_LIMITER_SLIM/INRUSH_CURRENT_LIMITER_SLIM.kicad_pcb (KiCad board)
At the start: 2 copper layers, 72 x 20 mm, 8 parts, among them J1 IN, J2 OUT

Commit message: renamed project
Other:
- board text added: "DIN RAIL INRUSH CURRENT LIMITER SLIM"
- board text removed: "DIN RAIL INRUSH CURRENT LIMIT SLIM"
Changed lines of the file:
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@@
     )
   )
-  (gr_text "DIN RAIL\nINRUSH CURRENT LIMIT SLIM" (at 137.795 101.6 -180) (layer F.SilkS)
+  (gr_text "DIN RAIL\nINRUSH CURRENT LIMITER SLIM" (at 138.303 101.981 -180) (layer F.SilkS)
     (effects (font (size 1 1) (thickness 0.15)))
   )

Commit message: silks adjusted
Other:
- board text added: "N L G"
- board text removed: "G L N"
Changed lines of the file:
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@@
     (descr "Varistor, diameter 12mm, width 3.9mm, pitch 7.5mm")
     (tags "varistor SIOV")
-    (fp_text reference RV2 (at 11.684 0.381 90) (layer F.SilkS)
+    (fp_text reference RV2 (at 11.684 0.381 270) (layer F.SilkS)
       (effects (font (size 1 1) (thickness 0.15)))
     )
@@
     (descr "Varistor, diameter 15.5mm, width 6.1mm, pitch 7.5mm")
     (tags "varistor SIOV")
-    (fp_text reference TH2 (at -6.583 3.937) (layer F.SilkS)
+    (fp_text reference TH2 (at -5.313 1.778 270) (layer F.SilkS)
       (effects (font (size 1 1) (thickness 0.15)))
     )
@@
     (descr "Varistor, diameter 21.5mm, width 5.3mm, pitch 10mm")
     (tags "varistor SIOV")
-    (fp_text reference TH1 (at -5.591 -3.683) (layer F.SilkS)
+    (fp_text reference TH1 (at -6.861 0.889 90) (layer F.SilkS)
       (effects (font (size 1 1) (thickness 0.15)))
     )
@@
     (descr "Terminal Block Phoenix MKDS-1,5-3-5.08, 3 pins, pitch 5.08mm, size 15.2x9.8mm^2, drill diamater 1.3mm, pad diameter 2.6mm, see http://www.farnell.com/datasheets/100425.pdf, script-generated using https://github.com/pointhi/kicad-footprint-generator/scripts/TerminalBlock_Phoenix")
     (tags "THT Terminal Block Phoenix MKDS-1,5-3-5.08 pitch 5.08mm size 15.2x9.8mm^2 drill 1.3mm pad 2.6mm")
-    (fp_text reference J2 (at -3.955 -0.546 90) (layer F.SilkS)
+    (fp_text reference J2 (at 14.079 -0.165 270) (layer F.SilkS)
       (effects (font (size 1 1) (thickness 0.15)))
     )
@@
     (descr "Terminal Block Phoenix MKDS-1,5-3-5.08, 3 pins, pitch 5.08mm, size 15.2x9.8mm^2, drill diamater 1.3mm, pad diameter 2.6mm, see http://www.farnell.com/datasheets/100425.pdf, script-generated using https://github.com/pointhi/kicad-footprint-generator/scripts/TerminalBlock_Phoenix")
     (tags "THT Terminal Block Phoenix MKDS-1,5-3-5.08 pitch 5.08mm size 15.2x9.8mm^2 drill 1.3mm pad 2.6mm")
-    (fp_text reference J1 (at -3.919 4.518 90) (layer F.SilkS)
+    (fp_text reference J1 (at -3.919 0.073 90) (layer F.SilkS)
       (effects (font (size 1 1) (thickness 0.15)))
     )
@@
     )
   )
+  (gr_text "N      L      G" (at 100.965 109.728 90) (layer F.SilkS)
+    (effects (font (size 1 1) (thickness 0.15)))
+  )
+  (gr_text "N      L     G" (at 170.942 110.363 90) (layer F.SilkS)
+    (effects (font (size 1 1) (thickness 0.15)))
+  )
   (gr_text "DIN RAIL\nINRUSH CURRENT LIMITER SLIM" (at 138.303 101.981 -180) (layer F.SilkS)
     (effects (font (size 1 1) (thickness 0.15)))
   )
-  (gr_text OUTPUT (at 167.259 119.126) (layer F.SilkS)
-    (effects (font (size 1 1) (thickness 0.15)))
-  )
-  (gr_text INPUT (at 104.013 119.126) (layer F.SilkS)
-    (effects (font (size 1 1) (thickness 0.15)))
-  )
-  (gr_text "G      L      N" (at 171.069 109.982 -90) (layer F.SilkS)
-    (effects (font (size 1 1) (thickness 0.15)))
-  )
-  (gr_text "G      L      N" (at 100.965 110.109 -90) (layer F.SilkS)
-    (effects (font (size 1 1) (thickness 0.15)))
-  )
+  (gr_text OUTPUT (at 167.259 100.965 -180) (layer F.SilkS)
+    (effects (font (size 1 1) (thickness 0.15)))
+  )
+  (gr_text INPUT (at 104.267 100.838 -180) (layer F.SilkS)
+    (effects (font (size 1 1) (thickness 0.15)))
+  )
