File: MODBUS_RTU_MIRROR/88x37x59mm/base/modbus_rtu_mirror_base_88x37x59mm.kicad_pcb (KiCad board)
At the start: 2 copper layers, 82 x 31 mm, 29 parts, among them J1 Conn_01x02_Female, J2 Conn_01x02_Female, J3 Conn_01x02_Female, J4 Conn_01x02_Female, J5 Conn_01x04_Male, J6 Conn_01x04_Male, U1 ST485EBDR, U2 ST485EBDR

Commit message: created folder for different processor version
Other:
- board text added: "MODBUS RTU MIRROR BASE BOARD"
- board text removed: "MODBUS RTU MIRROR BASE"
Changed lines of the file:
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@@
   )
   (paper "A4")
+  (title_block
+    (title "Modbus RTU mirror base board")
+  )
   (layers
     (0 "F.Cu" signal)
@@
   (gr_line (start 133 131) (end 133 129.5) (layer "Edge.Cuts") (width 0.1))
   (gr_line (start 149 100) (end 182 100) (layer "Edge.Cuts") (width 0.1))
-  (gr_text "MODBUS RTU MIRROR\nBASE" (at 113.157 101.6) (layer "B.SilkS")
+  (gr_text "MODBUS RTU MIRROR\nBASE BOARD" (at 113.157 101.6) (layer "B.SilkS")
     (effects (font (size 0.8 0.8) (thickness 0.2)) (justify left mirror))
   )
-  (gr_text "MODBUS RTU MIRROR\nBASE" (at 100.33 101.473) (layer "F.SilkS")
+  (gr_text "MODBUS RTU MIRROR\nBASE BOARD" (at 100.33 101.473) (layer "F.SilkS")
     (effects (font (size 0.8 0.8) (thickness 0.2)) (justify left))
   )
